Commit message: update-to-speed

File: bme_robot/urdf/bme.urdf (robot description, URDF)
Before this commit: robot bme, 8 links, 7 joints
Links:
- removed link kinect
- removed link motor_left
- removed link motor_right
- removed link support_wheel_left
- removed link support_wheel_right
- removed link wheel_left
- removed link wheel_right
- added link left_wheel; visual mesh filename=package://bme_robot/meshes/motor.STL scale=0.001 0.001 0.001
- added link right_wheel; visual mesh filename=package://bme_robot/meshes/motor.STL scale=0.001 0.001 0.001
Joints:
- removed joint base_link_to_kinect
- removed joint base_link_to_motor_left
- removed joint base_link_to_motor_right
- removed joint base_link_to_support_wheel_left
- removed joint base_link_to_support_wheel_right
- removed joint motor_left_to_wheel_left
- removed joint motor_right_to_wheel_right
- added joint left_joint: type fixed, parent base_link, child left_wheel, origin xyz=0 0.07 0.059
- added joint right_joint: type fixed, parent base_link, child right_wheel, origin xyz=0 -0.07 0.059
